Commit message: Add 3D model and launch with sensors

File: urdf/3dmodel_gz_control.xacro (robot description, xacro)
@@ -7,6 +7,6 @@
             <left_joint>left_wheel_joint</left_joint>
             <right_joint>right_wheel_joint</right_joint>
-            <wheel_separation>1.2</wheel_separation>
-            <wheel_radius>0.4</wheel_radius>
+            <wheel_separation>0.47</wheel_separation>
+            <wheel_radius>0.15</wheel_radius>
             <odom_publish_frequency>1</odom_publish_frequency>
             <topic>cmd_vel</topic>

File: urdf/laser.xacro (robot description, xacro)
@@ -2,8 +2,9 @@
 <robot xmlns:xacro="http://www.ros.org/wiki/xacro">
     <xacro:include filename="inertia_macro.xacro"/>
+<!--
     <joint name="laser_joint" type="fixed">
         <parent link="body_link"/>
         <child link="laser_frame"/>
-        <origin xyz="0.01 0 0.1" rpy="0 0 0"/>
+        <origin xyz="0.7 0 0.1" rpy="0 1.57 0"/>
     </joint>
     <link name="laser_frame">
@@ -24,4 +25,5 @@
         </xacro:inertial_cylinder>
     </link>
+-->
 <gazebo reference="laser_frame">
   <sensor name="laser" type="gpu_lidar">
@@ -35,11 +37,16 @@
       <scan>
         <horizontal>
+          <!--
           <samples>360</samples>
           <min_angle>-3.14</min_angle>
           <max_angle>3.14</max_angle>
+          -->
+          <samples>1</samples>
+          <min_angle>0</min_angle>
+          <max_angle>0</max_angle>
         </horizontal>
       </scan>
       <range>
-        <min>0.3</min>
+        <min>0.06</min>
         <max>12.0</max>
         <resolution>0.01</resolution>

File: urdf/lf_robot.urdf.xacro (robot description, xacro)
@@ -72,5 +72,5 @@
         <child link="right_wheel_link"/>
         <origin xyz="0.4 -0.275 0" rpy="${pi/2} 0 0"/>
-        <axis xyz="0 0 -1"/>
+        <axis xyz="0 0 1"/>
     </joint>
     <!--LEFT WHEEL LINK-->
@@ -125,3 +125,25 @@
         <origin xyz="-0.15 0 0" rpy="0 0 0"/>
     </joint>
+        <joint name="laser_joint" type="fixed">
+        <parent link="body_link"/>
+        <child link="laser_frame"/>
+        <origin xyz="0.7 0 0.1" rpy="0 1.57 0"/>
+    </joint>
+    <link name="laser_frame">
+        <visual>
+            <origin xyz="0 0 0"/>
+            <geometry>
+                <cylinder radius="0.05" length="0.03"/>
+            </geometry>
+        </visual>
+        <collision>
+            <origin xyz="0 0 0"/>
+            <geometry>
+                <cylinder radius="0.05" length="0.03"/>
+            </geometry>
+        </collision>
+        <xacro:inertial_cylinder mass="0.1" radius="0.05" length="0.03">
+            <origin xyz="0 0 0" rpy="0 0 0"/>
+        </xacro:inertial_cylinder>
+    </link>
 </robot>

File: urdf/robot.xacro (robot description, xacro)
@@ -2,3 +2,5 @@
 <robot xmlns:xacro="http://www.ros.org/wiki/xacro" name="line_following_robot">
     <xacro:include filename="lf_robot.urdf.xacro" />
+    <xacro:include filename="laser.xacro" />
+    <xacro:include filename="3dmodel_gz_control.xacro" />
 </robot>
